File: Hardware/e_book_reader.brd (EAGLE design)
At the start: 171.3 x 111.8 mm, 103 parts, among them IC1 BD5229G-TR, IC4 XC6220A331MR-G, J1 FH34SRJ-24S-0.5SH_99_, J2 SAMACSYS_PARTS_USB4110-GF-A, J3 QWIIC_RIGHT_ANGLE, J4 112A-TAAR-R03_ATTEND, Q1 ESP32_WROVER_SPARKFUN-DISCRET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, Q2 ESP32_WROVER_SPARKFUN-DISCRET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, Q3 SI1308EDL-T1-GE3, U1 W25Q512JVEIQ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

Commit message: fixed issues
Parts:
- D10, D11, D12, D6, D8, D9: value PGB1010603MRPGB1010603MR -> PGB1010603MR
- D3, D4, D5: value MBR0530MY_MBR -> MBR0530
- moved U2 0.12 mm to (12.5, 39.6)
Routing:
- net SCK: track 193.8 -> 222.3 mm, vias 7 -> 6
- net RESE: track 24.4 -> 39.7 mm, vias 2 -> 0
- net SCL: track 211.4 -> 196.7 mm
- net USB_D-: track 132.4 -> 146.8 mm, vias 4 -> 2
- net EPD_RST: track 124.3 -> 109.9 mm, vias 4 -> 3
- net N$6: track 22.9 -> 36.8 mm, vias 2 -> 0
- net 3V3: track 435.7 -> 446.0 mm, vias 6 -> 4
- net FLASH_CS: track 40.4 -> 48.9 mm, vias 3 -> 4
- net EPD_CS: track 185.7 -> 177.9 mm, vias 6 -> 8
- net EPD_3V3: track 97.0 -> 89.3 mm, vias 4 -> 5
- net USB_D+: track 131.9 -> 139.5 mm
- net N$13: track 24.4 -> 16.9 mm, vias 0 -> 2
- net RESE': track 25.5 -> 19.9 mm, vias 0 -> 2
- net GND: track 641.3 -> 646.8 mm, vias 7 -> 46
- net INT_RTC: track 95.1 -> 89.7 mm, vias 5 -> 2
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Other:
- outline, holes or cut-outs redrawn
- board text added: "3V3"
- board text added: "BME688"
- board text added: "BOOT_BUTTON"
- board text added: "C10"
- board text added: "C10_SUPERCAP"
- board text added: "C1_BAT"
- board text added: "C1_BAT1"
- board text added: "C1_BAT2"
- board text added: "C2"
- board text added: "C2_BAT"
- board text added: "C3"
- board text added: "C4"
- board text added: "C4_USB"
- board text added: "C5"
- board text added: "C5_USB"
- board text added: "C6"
- board text added: "C8"
- board text added: "C9"
- board text added: "CHANGE_BUTTON"
- board text added: "CHG_LED"
- board text added: "C_DELAY"
- board text added: "D1"
- board text added: "D10"
- board text added: "D11"
- board text added: "D12"
- board text added: "D6"
- board text added: "D8"
- board text added: "D9"
- board text added: "DS3231SN#"
- board text added: "EPD_3V3"
- board text added: "EPD_3V3_C"
- board text added: "EPD_BUSY"
- board text added: "EPD_C1"
- board text added: "EPD_C10"
- board text added: "EPD_C11"
- board text added: "EPD_C12"
- board text added: "EPD_C2"
- board text added: "EPD_C5"
- board text added: "EPD_C6"
- board text added: "EPD_C7"
- board text added: "EPD_C8"
- board text added: "EPD_C9"
- board text added: "EPD_CS"
- board text added: "EPD_DC"
- board text added: "EPD_RST"
- board text added: "GND"
- board text added: "IC1"
- board text added: "IC4"
- board text added: "INT_RTC"
- board text added: "L1"
- board text added: "MCP73831"
- board text added: "MISO"
- board text added: "MOSFET"
- board text added: "MOSI"
- board text added: "PFMF.050.1"
- board text added: "QWIIC_RIGHT_ANGLE"
- board text added: "R1"
- board text added: "R1-PINH"
- board text added: "R10"
- board text added: "R1_BAT"
- board text added: "R1_PINH1"
- board text added: "R1_PWRUSB"
- board text added: "R2"
- board text added: "R2-PINH"
- board text added: "R2-PINH1"
- board text added: "R2-USB"
- board text added: "R2_BAT"
- board text added: "R5"
- board text added: "R6"
- board text added: "R7"
- board text added: "R8"
- board text added: "R9"
- board text added: "RESET_BUTTON"
- board text added: "RX"
- board text added: "R_BOOT"
- board text added: "R_CAPACITOR"
- board text added: "R_CHANGE"
- board text added: "R_CL1"
- board text added: "R_J2"
- board text added: "R_RESET"
- board text added: "SCK"
- board text added: "SJ"
- board text added: "TX"
- board text added: "USB"
- board text added: "VBAT"
- board text added: "VBUS"
- board text added: "W25Q512JVEIQ"
