File: Hardware/e_book_reader.sch (EAGLE design)
At the start: 103 parts, among them IC1 BD5229G-TR, IC4 XC6220A331MR-G, J1 FH34SRJ-24S-0.5SH_99_, J2 SAMACSYS_PARTS_USB4110-GF-A, J3 QWIIC_RIGHT_ANGLE, J4 112A-TAAR-R03_ATTEND, Q1 ESP32_WROVER_SPARKFUN-DISCRET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, Q2 ESP32_WROVER_SPARKFUN-DISCRET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, Q3 SI1308EDL-T1-GE3, U1 W25Q512JVEIQ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

Commit message: fixed issues
Parts:
- D10, D11, D12, D6, D8, D9: value PGB1010603MRPGB1010603MR -> PGB1010603MR
- D3, D4, D5: value MBR0530MY_MBR -> MBR0530
Other:
- moved on the sheet: C2, C4, R1-PINH, R2-PINH
